File: Chapter_1/Multimeter/multimeter.kicad_pcb (KiCad board)
At the start: 2 copper layers, 17 parts, among them Q1 BC557, Q10 BC557, Q11 BC557, Q12 BC557, Q13 BC557, Q14 IRLZ44N, Q15 BC557, Q16 BC557, Q2 BC557, Q21 IRLZ44N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

Commit message: continuing layout
Parts:
- removed Q1, Q10, Q11, Q12, Q13, Q15, Q16, Q2, Q3, Q4, Q5, Q6, Q7, Q8, Q9: BC557, Package_TO_SOT_THT:TO-92_Inline
- removed Q14, Q21: IRLZ44N, Package_TO_SOT_THT:TO-220-3_Vertical
- added D3: RED - LED, LED_THT:LED_D1.8mm_W3.3mm_H2.4mm, F.Cu at (163.2, 59.3)
- added D4: GREEN - LED, LED_THT:LED_D1.8mm_W3.3mm_H2.4mm, F.Cu at (69.0, 39.0)
- added D5: WHITE- LED, LED_THT:LED_D1.8mm_W3.3mm_H2.4mm, F.Cu at (176.7, 59.3)
- added D6: 1N4148WT, Diode_THT:D_5W_P12.70mm_Horizontal, F.Cu at (146.2, 47.0)
- added D7: 1N4148WT, Diode_THT:D_5W_P12.70mm_Horizontal, F.Cu at (122.3, 79.3)
- added J1: Screw_Terminal_01x02, Connector_PinSocket_2.54mm:PinSocket_1x02_P2.54mm_Vertical, F.Cu at (215.4, 77.0)
- added J2: Conn_01x02_Socket, Connector_PinSocket_2.54mm:PinSocket_1x02_P2.54mm_Vertical, F.Cu at (220.0, 77.0)
- added Q17: BC547, Package_TO_SOT_THT:TO-92_Inline, F.Cu at (83.3, 97.0)
- added Q18: BC547, Package_TO_SOT_THT:TO-92_Inline, F.Cu at (83.2, 103.0)
- added Q19: BC547, Package_TO_SOT_THT:TO-92_Inline, F.Cu at (91.3, 90.2)
- added Q20: BC547, Package_TO_SOT_THT:TO-92_Inline, F.Cu at (82.1, 70.2)
- added Q22: BC547, Package_TO_SOT_THT:TO-92_Inline, F.Cu at (82.1, 76.2)
- added Q23: BC547, Package_TO_SOT_THT:TO-92_Inline, F.Cu at (91.5, 64.0)
- added Q24: BC547, Package_TO_SOT_THT:TO-92_Inline, F.Cu at (121.0, 63.0)
- added Q25: BC547, Package_TO_SOT_THT:TO-92_Inline, F.Cu at (121.0, 69.0)
- added Q26: BC547, Package_TO_SOT_THT:TO-92_Inline, F.Cu at (130.3, 52.5)
- added Q27: BC547, Package_TO_SOT_THT:TO-92_Inline, F.Cu at (116.5, 104.7)
- added Q28: BC547, Package_TO_SOT_THT:TO-92_Inline, F.Cu at (116.5, 111.0)
- added Q29: BC547, Package_TO_SOT_THT:TO-92_Inline, F.Cu at (122.3, 97.0)
- added Q30: BC547, Package_TO_SOT_THT:TO-92_Inline, F.Cu at (152.3, 105.5)
- added Q31: BC547, Package_TO_SOT_THT:TO-92_Inline, F.Cu at (152.5, 111.7)
- added Q32: BC547, Package_TO_SOT_THT:TO-92_Inline, F.Cu at (159.5, 98.2)
- added Q33: IRLZ44N, Package_TO_SOT_THT:TO-220-3_Vertical, F.Cu at (147.0, 59.0)
- added Q34: IRLZ44N, Package_TO_SOT_THT:TO-220-3_Vertical, F.Cu at (180.0, 83.5)
- added R1: 10K, Resistor_THT:R_Axial_DIN0309_L9.0mm_D3.2mm_P12.70mm_Horizontal, F.Cu at (63.5, 98.0)
- added R10: 10K, Resistor_THT:R_Axial_DIN0309_L9.0mm_D3.2mm_P12.70mm_Horizontal, F.Cu at (63.3, 71.5)
- added R11: 10K, Resistor_THT:R_Axial_DIN0309_L9.0mm_D3.2mm_P12.70mm_Horizontal, F.Cu at (63.1, 77.5)
- added R12: 1K, Resistor_THT:R_Axial_DIN0309_L9.0mm_D3.2mm_P12.70mm_Horizontal, F.Cu at (63.1, 65.5)
- added R13: 1K, Resistor_THT:R_Axial_DIN0309_L9.0mm_D3.2mm_P12.70mm_Horizontal, F.Cu at (75.7, 58.5)
- added R14: 1K, Resistor_THT:R_Axial_DIN0309_L9.0mm_D3.2mm_P12.70mm_Horizontal, F.Cu at (163.5, 65.0)
- added R15: 1K, Resistor_THT:R_Axial_DIN0309_L9.0mm_D3.2mm_P12.70mm_Horizontal, F.Cu at (73.3, 39.0)
- added R16: 10K, Resistor_THT:R_Axial_DIN0309_L9.0mm_D3.2mm_P12.70mm_Horizontal, F.Cu at (103.2, 64.0)
- added R17: 10K, Resistor_THT:R_Axial_DIN0309_L9.0mm_D3.2mm_P12.70mm_Horizontal, F.Cu at (103.2, 70.0)
- added R18: 1K, Resistor_THT:R_Axial_DIN0309_L9.0mm_D3.2mm_P12.70mm_Horizontal, F.Cu at (103.2, 57.5)
- added R19: 1K, Resistor_THT:R_Axial_DIN0309_L9.0mm_D3.2mm_P12.70mm_Horizontal, F.Cu at (110.7, 49.0)
- added R20: 10K, Resistor_THT:R_Axial_DIN0309_L9.0mm_D3.2mm_P12.70mm_Horizontal, F.Cu at (96.2, 106.0)
- added R21: 10K, Resistor_THT:R_Axial_DIN0309_L9.0mm_D3.2mm_P12.70mm_Horizontal, F.Cu at (96.5, 112.0)
- added R22: 1K, Resistor_THT:R_Axial_DIN0309_L9.0mm_D3.2mm_P12.70mm_Horizontal, F.Cu at (96.2, 101.0)
- added R23: 1K, Resistor_THT:R_Axial_DIN0309_L9.0mm_D3.2mm_P12.70mm_Horizontal, F.Cu at (104.7, 92.5)
- added R24: 10K, Resistor_THT:R_Axial_DIN0309_L9.0mm_D3.2mm_P12.70mm_Horizontal, F.Cu at (134.7, 107.0)
- added R25: 10K, Resistor_THT:R_Axial_DIN0309_L9.0mm_D3.2mm_P12.70mm_Horizontal, F.Cu at (134.7, 113.0)
- added R26: 1K, Resistor_THT:R_Axial_DIN0309_L9.0mm_D3.2mm_P12.70mm_Horizontal, F.Cu at (134.7, 100.5)
- added R27: 1K, Resistor_THT:R_Axial_DIN0309_L9.0mm_D3.2mm_P12.70mm_Horizontal, F.Cu at (143.2, 94.0)
- added R28: 1K, Resistor_THT:R_Axial_DIN0309_L9.0mm_D3.2mm_P12.70mm_Horizontal, F.Cu at (175.8, 51.5)
- added R29: 5K, Resistor_THT:R_Axial_DIN0309_L9.0mm_D3.2mm_P12.70mm_Horizontal, F.Cu at (154.5, 76.3)
- added R30: 1_Ohm, Resistor_THT:R_Axial_DIN0309_L9.0mm_D3.2mm_P12.70mm_Horizontal, F.Cu at (163.3, 88.5)
- added R31: 5K, Resistor_THT:R_Axial_DIN0309_L9.0mm_D3.2mm_P12.70mm_Horizontal, F.Cu at (146.5, 63.1)
- added R32: 5K, Resistor_THT:R_Axial_DIN0309_L9.0mm_D3.2mm_P12.70mm_Horizontal, F.Cu at (175.8, 83.0)
- added R7: 1K, Resistor_THT:R_Axial_DIN0309_L9.0mm_D3.2mm_P12.70mm_Horizontal, F.Cu at (63.3, 91.5)
- added R8: 10K, Resistor_THT:R_Axial_DIN0309_L9.0mm_D3.2mm_P12.70mm_Horizontal, F.Cu at (63.5, 103.5)
- added R9: 1K, Resistor_THT:R_Axial_DIN0309_L9.0mm_D3.2mm_P12.70mm_Horizontal, F.Cu at (74.8, 86.5)

Commit message: final
Parts:
- added Q1: IRLZ44N, Package_TO_SOT_THT:TO-220-3_Vertical, F.Cu at (166.7, 56.2)
- added R2: 5K, Resistor_THT:R_Axial_DIN0309_L9.0mm_D3.2mm_P12.70mm_Horizontal, F.Cu at (169.4, 62.0)
- added SW1: SW_DPST_x2, Button_Switch_THT:SW_DIP_SPSTx01_Piano_10.8x4.1mm_W7.62mm_P2.54mm, F.Cu at (46.1, 95.0)
- added SW2: SW_DPST_x2, Button_Switch_THT:SW_DIP_SPSTx01_Piano_10.8x4.1mm_W7.62mm_P2.54mm, F.Cu at (46.1, 103.2)
- added SW3: SW_DPST_x2, Button_Switch_THT:SW_DIP_SPSTx01_Piano_10.8x4.1mm_W7.62mm_P2.54mm, F.Cu at (46.3, 71.2)
- J1: footprint Connector_PinSocket_2.54mm:PinSocket_1x02_P2.54mm_Vertical -> TerminalBlock:TerminalBlock_Xinya_XY308-2.54-2P_1x02_P2.54mm_Horizontal
- moved J2 60.1 mm to (171.8, 112.8), turned to 90 degrees
- moved J1 33.5 mm to (182.4, 71.5), turned to -90 degrees
- moved R14 23.8 mm to (155.8, 42.5)
- moved D3 22.6 mm to (151.8, 39.8)
- moved D5 22.1 mm to (173.0, 37.5), turned to -90 degrees
- moved R28 16.0 mm to (168.5, 37.2)
- moved R19 3.28 mm to (108.0, 51.0)
- moved D6 3.28 mm to (143.6, 49.0)
- moved Q26 3.28 mm to (127.8, 54.5)
Connections:
- Q33 pad 1: /SIGNAL_MEASURING_AMPS -> /SIGNAL_MEASURING_VOLTS
- Q34 pad 1: /SIGNAL_MEASURING_VOLTS -> /SIGNAL_MEASURING_AMPS
- R31 pad 1: /SIGNAL_MEASURING_AMPS -> /SIGNAL_MEASURING_VOLTS
- R32 pad 1: /SIGNAL_MEASURING_VOLTS -> /SIGNAL_MEASURING_AMPS
Routing:
- net VCC: track 0.00 -> 228.4 mm, vias 0 -> 8
- net /SIGNAL_POWER_BUTTON: track 0.00 -> 192.0 mm
- net Net-(D5-A): track 0.00 -> 129.1 mm
- net Net-(D6-K): track 0.00 -> 121.3 mm
- net /SIGNAL_MEASURING_AMPS: track 0.00 -> 104.0 mm, vias 0 -> 2
- net /INPUT_POSITIVE: track 0.00 -> 81.3 mm, vias 0 -> 2
- net /SIGNAL_NOT_ALLOWED: track 0.00 -> 75.0 mm
- net /NAND_OUTPUT: track 0.00 -> 73.4 mm
- net /SIGNAL_AMMETER: track 0.00 -> 69.8 mm, vias 0 -> 2
- net /SIGNAL_MEASURING_VOLTS: track 0.00 -> 60.8 mm
- net Net-(J1-Pin_1): track 0.00 -> 59.5 mm, vias 0 -> 2
- net /INPUT_NEGATIVE: track 0.00 -> 49.8 mm
- net /SIGNAL_VOLTMETER: track 0.00 -> 46.0 mm
- net /SIGNAL_DUAL-METER: track 0.00 -> 33.8 mm
- net Net-(Q27-C): track 0.00 -> 19.8 mm
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- added copper zone on B.Cu, net GND
Other:
- board outline added: 148.8 x 87.8 mm
