File: Chapter_1/Multimeter/_autosave-multimeter.kicad_pcb (KiCad board)
At the start: 2 copper layers, 148.8 x 87.8 mm, 56 parts, among them J1 Screw_Terminal_01x02, J2 Conn_01x02_Socket, Q1 IRLZ44N, Q17 BC547, Q18 BC547, Q19 BC547, Q20 BC547, Q22 BC547, Q23 BC547, Q24 BC547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

Commit message: -
Parts:
- moved R14 1.25 mm to (155.9, 43.8)
Changed lines of the file:
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@@
 	(footprint "Resistor_THT:R_Axial_DIN0309_L9.0mm_D3.2mm_P12.70mm_Horizontal"
 		(layer "F.Cu")
-		(at 155.8 42.5)
+		(at 155.9 43.75)
 		(descr "Resistor, Axial_DIN0309 series, Axial, Horizontal, pin pitch=12.7mm, 0.5W = 1/2W, length*diameter=9*3.2mm^2, http://cdn-reichelt.de/documents/datenblatt/B400/1_4W%23YAG.pdf")
 		(tags "Resistor Axial_DIN0309 series Axial Horizontal pin pitch 12.7mm 0.5W = 1/2W length 9mm diameter 3.2mm")
